File: blinds_motor_driver.sch (KiCad schematic (older format))
At the start: 6 parts, among them J1 Barrel_Jack, J2 Screw_Terminal_01x04, U1 LM2596_HW411, U2 WeMos_D1_mini

Commit message: Box schematic
Other:
- note added: "ESP8266"
- note added: "Stepper Driver"
- note added: "Voltage Regulator"
- moved on the sheet: A1, C3, J2, U2
